File: nfc_edit.sch (EAGLE design)
At the start: 5 parts

Commit message: .2uF capacitor has been added
NFC added and connected via power only (no data transfer with ATTiny85)
Parts:
- added C1: 0.2uf, SparkFun-Capacitors:CAP1206
Connections:
- net 2.8V: now also C1.1
Changed lines of the file:
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@@
 <part name="SJ1" library="microbuilder" deviceset="SOLDERJUMPER" device=""/>
 <part name="U1" library="AlterNail" deviceset="NT3H1101" device=""/>
+<part name="C1" library="SparkFun-Capacitors" deviceset="CAP" device="1206" value="0.2uf"/>
 </parts>
 <sheets>
@@
 <instance part="SJ1" gate="1" x="73.66" y="12.7"/>
 <instance part="U1" gate="G$1" x="12.7" y="20.32" rot="R180"/>
+<instance part="C1" gate="G$1" x="35.56" y="20.32"/>
 </instances>
 <busses>
@@
 <segment>
 <pinref part="MCU" gate="G$1" pin="GND"/>
-<wire x1="25.4" y1="15.24" x2="40.64" y2="15.24" width="0.1524" layer="91"/>
+<wire x1="25.4" y1="15.24" x2="35.56" y2="15.24" width="0.1524" layer="91"/>
 <label x="33.02" y="15.24" size="1.778" layer="95"/>
+<wire x1="35.56" y1="15.24" x2="40.64" y2="15.24" width="0.1524" layer="91"/>
+<wire x1="35.56" y1="20.32" x2="35.56" y2="15.24" width="0.1524" layer="91"/>
+<junction x="35.56" y="15.24"/>
 </segment>
 <segment>
@@
 <segment>
 <pinref part="MCU" gate="G$1" pin="VCC"/>
-<wire x1="40.64" y1="27.94" x2="27.94" y2="27.94" width="0.1524" layer="91"/>
-<label x="33.02" y="27.94" size="1.778" layer="95"/>
+<wire x1="40.64" y1="27.94" x2="35.56" y2="27.94" width="0.1524" layer="91"/>
+<label x="33.02" y="33.02" size="1.778" layer="95"/>
 <pinref part="U1" gate="G$1" pin="V_OUT"/>
+<wire x1="35.56" y1="27.94" x2="27.94" y2="27.94" width="0.1524" layer="91"/>
 <wire x1="27.94" y1="27.94" x2="25.4" y2="27.94" width="0.1524" layer="91"/>
+<pinref part="C1" gate="G$1" pin="1"/>
+<wire x1="35.56" y1="25.4" x2="35.56" y2="27.94" width="0.1524" layer="91"/>
+<junction x="35.56" y="27.94"/>
 </segment>
 </net>
