File: nfc_with_data_transfer_no_accel_2.0.sch (EAGLE design)
At the start: 7 parts

Commit message: fixed rst
Connections:
- net DOT1: now also MCU.PB1(MISO); no longer MCU.PB3(ADC3)
- net DOT5: now also MCU.PB5(NRES); no longer MCU.PB1(MISO)
- net RST: now also MCU.PB3(ADC3); no longer MCU.PB5(NRES)
Changed lines of the file:
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@@
 </segment>
 <segment>
-<pinref part="MCU" gate="G$1" pin="PB3(ADC3)"/>
-<wire x1="71.12" y1="20.32" x2="76.2" y2="20.32" width="0.1524" layer="91"/>
-<label x="71.12" y="20.32" size="1.778" layer="95"/>
+<pinref part="MCU" gate="G$1" pin="PB1(MISO)"/>
+<wire x1="71.12" y1="25.4" x2="76.2" y2="25.4" width="0.1524" layer="91"/>
+<label x="71.12" y="25.4" size="1.778" layer="95"/>
 </segment>
 </net>
@@
 </segment>
 <segment>
-<pinref part="MCU" gate="G$1" pin="PB5(NRES)"/>
-<wire x1="71.12" y1="15.24" x2="76.2" y2="15.24" width="0.1524" layer="91"/>
-<label x="71.12" y="15.24" size="1.778" layer="95"/>
+<pinref part="MCU" gate="G$1" pin="PB3(ADC3)"/>
+<wire x1="71.12" y1="20.32" x2="76.2" y2="20.32" width="0.1524" layer="91"/>
+<label x="71.12" y="20.32" size="1.778" layer="95"/>
 </segment>
 </net>
@@
 </segment>
 <segment>
-<pinref part="MCU" gate="G$1" pin="PB1(MISO)"/>
-<wire x1="71.12" y1="25.4" x2="76.2" y2="25.4" width="0.1524" layer="91"/>
-<label x="71.12" y="25.4" size="1.778" layer="95"/>
+<pinref part="MCU" gate="G$1" pin="PB5(NRES)"/>
+<wire x1="71.12" y1="15.24" x2="76.2" y2="15.24" width="0.1524" layer="91"/>
+<label x="71.12" y="15.24" size="1.778" layer="95"/>
 </segment>
 </net>

Commit message: final
Connections:
- removed net DOT3: EINK.5, MCU.PB4(ADC2)
- net DOT1: now also MCU.PB4(ADC2); no longer MCU.PB1(MISO)
- net DOT5: now also MCU.PB1(MISO); no longer MCU.PB5(NRES)
- net GND: now also EINK.5
Changed lines of the file:
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@@
 </busses>
 <nets>
-<net name="DOT3" class="0">
-<segment>
-<pinref part="EINK" gate="A" pin="5"/>
-<wire x1="134.62" y1="10.16" x2="142.24" y2="10.16" width="0.1524" layer="91"/>
-<label x="137.16" y="10.16" size="1.778" layer="95"/>
-</segment>
-<segment>
-<pinref part="MCU" gate="G$1" pin="PB4(ADC2)"/>
-<wire x1="71.12" y1="17.78" x2="76.2" y2="17.78" width="0.1524" layer="91"/>
-<label x="71.12" y="17.78" size="1.778" layer="95"/>
-</segment>
-</net>
 <net name="DOT1" class="0">
 <segment>
@@
 </segment>
 <segment>
-<pinref part="MCU" gate="G$1" pin="PB1(MISO)"/>
-<wire x1="71.12" y1="25.4" x2="76.2" y2="25.4" width="0.1524" layer="91"/>
-<label x="71.12" y="25.4" size="1.778" layer="95"/>
+<pinref part="MCU" gate="G$1" pin="PB4(ADC2)"/>
+<wire x1="71.12" y1="17.78" x2="76.2" y2="17.78" width="0.1524" layer="91"/>
+<label x="71.12" y="17.78" size="1.778" layer="95"/>
 </segment>
 </net>
@@
 </segment>
 <segment>
-<pinref part="MCU" gate="G$1" pin="PB5(NRES)"/>
-<wire x1="71.12" y1="15.24" x2="76.2" y2="15.24" width="0.1524" layer="91"/>
-<label x="71.12" y="15.24" size="1.778" layer="95"/>
+<pinref part="MCU" gate="G$1" pin="PB1(MISO)"/>
+<wire x1="71.12" y1="25.4" x2="76.2" y2="25.4" width="0.1524" layer="91"/>
+<label x="71.12" y="25.4" size="1.778" layer="95"/>
 </segment>
 </net>
@@
 <wire x1="33.02" y1="17.78" x2="33.02" y2="15.24" width="0.1524" layer="91"/>
 </segment>
+<segment>
+<pinref part="EINK" gate="A" pin="5"/>
+<wire x1="134.62" y1="10.16" x2="142.24" y2="10.16" width="0.1524" layer="91"/>
+<label x="137.16" y="10.16" size="1.778" layer="95"/>
+</segment>
 </net>
